File: KiCAD/KZ80_PIOSIO.kicad_pcb (KiCad board)
At the start: 2 copper layers, 100 x 75 mm, 33 parts, among them J1 CON-A, J2 CON-B, J3 PIO-A, J4 PIO-B, J5 SBC8080 BUS, J6 SPK_JP, J7 ADDR-JP, J8 Z80 CONTROL, Q1 2SC1815, U1 Z80-SIO2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

Commit message: シルク見直し。ガーバーデータ再出力
Other:
- board text added: "NC"
- board text added: "~BUSA"
- board text added: "~BUSR"
- board text added: "~HALT"
- board text added: "~INT"
- board text added: "~IORQ"
- board text added: "~M1"
- board text added: "~MRQ"
- board text added: "~NMI"
- board text added: "~RD"
- board text added: "~RES"
- board text added: "~RFSH"
- board text added: "~WAIT"
- board text added: "~WR"
Changed lines of the file:
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@@
   (general
     (thickness 1.6)
-    (drawings 38)
+    (drawings 52)
     (tracks 1158)
     (zones 0)
@@
     )
   )
+  (gr_text ~HALT (at 188.8 67.8) (layer B.SilkS)
+    (effects (font (size 1 1) (thickness 0.15)) (justify mirror))
+  )
+  (gr_text ~RFSH (at 188.609523 65.2) (layer B.SilkS)
+    (effects (font (size 1 1) (thickness 0.15)) (justify mirror))
+  )
+  (gr_text ~NMI (at 189.204761 62.6) (layer B.SilkS)
+    (effects (font (size 1 1) (thickness 0.15)) (justify mirror))
+  )
+  (gr_text ~BUSR (at 188.538095 60) (layer B.SilkS)
+    (effects (font (size 1 1) (thickness 0.15)) (justify mirror))
+  )
+  (gr_text ~M1 (at 189.490476 57.6) (layer B.SilkS)
+    (effects (font (size 1 1) (thickness 0.15)) (justify mirror))
+  )
+  (gr_text ~IORQ (at 188.75238 55.2) (layer B.SilkS)
+    (effects (font (size 1 1) (thickness 0.15)) (justify mirror))
+  )
+  (gr_text ~RD (at 189.538095 51.2) (layer B.SilkS)
+    (effects (font (size 1 1) (thickness 0.15)) (justify mirror))
+  )
+  (gr_text NC (at 196.895238 67.8) (layer B.SilkS)
+    (effects (font (size 1 1) (thickness 0.15)) (justify mirror))
+  )
+  (gr_text ~WAIT (at 197.490476 65.4) (layer B.SilkS)
+    (effects (font (size 1 1) (thickness 0.15)) (justify mirror))
+  )
+  (gr_text ~INT (at 197.014286 62.8) (layer B.SilkS)
+    (effects (font (size 1 1) (thickness 0.15)) (justify mirror))
+  )
+  (gr_text ~BUSA (at 197.8 60.2) (layer B.SilkS)
+    (effects (font (size 1 1) (thickness 0.15)) (justify mirror))
+  )
+  (gr_text ~RES (at 197.3 57.6) (layer B.SilkS)
+    (effects (font (size 1 1) (thickness 0.15)) (justify mirror))
+  )
+  (gr_text ~MRQ (at 197.466667 55) (layer B.SilkS)
+    (effects (font (size 1 1) (thickness 0.15)) (justify mirror))
+  )
+  (gr_text ~WR (at 196.942857 52.8) (layer B.SilkS)
+    (effects (font (size 1 1) (thickness 0.15)) (justify mirror))
+  )
   (gr_text 4060 (at 170.2 63.8 90) (layer F.SilkS)
