File: exsample/I2C-PPI/I2C-PPI.sch (KiCad schematic (older format))
At the start: 7 parts, among them J1 PPI CON-A, J2 PPI CON-B, J3 I2C RTC(DS3231)

Commit message: PPI-I2C回路図修正
Connections:
- net PB0 renamed PC0
- net PB1 renamed PC4
Changed lines of the file:
@@
 	6550 3700 7200 3700
 Text GLabel 5400 3600 0    50   BiDi ~ 0
-PB0
+PC0
 Text GLabel 5400 3800 0    50   BiDi ~ 0
-PB1
+PC4
 NoConn ~ 3950 3950
 NoConn ~ 3950 4050
